Commit message: updated manipulator base position

File: model_changes/turtlebot3_manipulation_robot.urdf.xacro (robot description, xacro)
@@ -7,5 +7,5 @@
   <!-- Base fixed joint -->
   <joint name="base_fixed" type="fixed">
-    <origin xyz="-0.1 0.0 0.135" rpy="0 0 0"/>
+    <origin xyz="-0.01 0.0 0.135" rpy="0 0 0"/>
     <parent link="base_link"/>
     <child link="link1"/>
