Commit message: Updated the model to more accurately represent the robot and fixed wheel position

File: model_changes/turtlebot3_waffle_pi_for_open_manipulator.urdf.xacro (robot description, xacro)
@@ -18,5 +18,5 @@
     </visual>
     <collision>
-      <origin xyz="-0.064 0 0.047" rpy="0 0 0"/>
+      <origin xyz="0.0 0 0.047" rpy="0 0 0"/>
       <geometry>
         <box size="0.266 0.266 0.094"/>
@@ -34,8 +34,21 @@
     </inertial>
   </link>
+  <joint name="manipulator_base_joint" type="fixed">
+    <parent link="base_link"/>
+    <child link="manipulator_base_link"/>
+    <origin xyz="0 0 0.131"/>
+  </joint>
+  <link name="manipulator_base_link">
+    <collision>
+      <origin xyz="0 0 0" rpy="0 0 0"/>
+      <geometry>
+        <box size="0.133 0.133 0.01"/>
+      </geometry>
+    </collision>
+  </link>
   <joint name="wheel_left_joint" type="continuous">
     <parent link="base_link"/>
     <child link="wheel_left_link"/>
-    <origin xyz="0.0 0.144 0.023" rpy="-1.57 0 0"/>
+    <origin xyz="0.064 0.144 0.023" rpy="-1.57 0 0"/>
     <axis xyz="0 0 1"/>
   </joint>
@@ -65,5 +78,5 @@
     <parent link="base_link"/>
     <child link="wheel_right_link"/>
-    <origin xyz="0.0 -0.144 0.023" rpy="-1.57 0 0"/>
+    <origin xyz="0.064 -0.144 0.023" rpy="-1.57 0 0"/>
     <axis xyz="0 0 1"/>
   </joint>
@@ -93,5 +106,5 @@
     <parent link="base_link"/>
     <child link="caster_back_right_link"/>
-    <origin xyz="-0.177 -0.064 -0.004" rpy="-1.57 0 0"/>
+    <origin xyz="-0.113 -0.064 -0.004" rpy="-1.57 0 0"/>
   </joint>
   <link name="caster_back_right_link">
@@ -113,5 +126,5 @@
     <parent link="base_link"/>
     <child link="caster_back_left_link"/>
-    <origin xyz="-0.177 0.064 -0.004" rpy="-1.57 0 0"/>
+    <origin xyz="-0.113 0.064 -0.004" rpy="-1.57 0 0"/>
   </joint>
   <link name="caster_back_left_link">
@@ -164,13 +177,20 @@
   </link>
   <joint name="camera_joint" type="fixed">
-    <origin xyz="0.073 -0.011 0.084" rpy="0 0 0"/>
+    <origin xyz="0.137 0 0.08" rpy="0 0 0"/>
     <parent link="base_link"/>
     <child link="camera_link"/>
   </joint>
   <link name="camera_link">
-    <collision>
-      <origin xyz="0.005 0.011 0.013" rpy="0 0 0"/>
-      <geometry>
-        <box size="0.015 0.030 0.027"/>
+    <visual>
+      <origin xyz="0 0 0" rpy="0 0 0"/>
+      <geometry>
+        <box size="0.02 0.08 0.02"/>
+      </geometry>
+      <material name="blue"/>
+    </visual>
+    <collision>
+      <origin xyz="0 0 0" rpy="0 0 0"/>
+      <geometry>
+        <box size="0.02 0.08 0.02"/>
       </geometry>
     </collision>
